Commit message: update humble-matterport

File: src/vehicle_simulator/urdf/lidar.urdf.xacro (robot description, xacro)
@@ -3,5 +3,5 @@
   <link name="lidar" />
   <xacro:include filename="$(find velodyne_description)/urdf/VLP-16.urdf.xacro"/>
-  <xacro:VLP-16 parent="lidar" name="velodyne" topic="/velodyne_points" hz="6.3" samples="350" min_range="0.1">
+  <xacro:VLP-16 parent="lidar" name="velodyne" topic="/velodyne_points" hz="6.3" samples="350" min_range="0.01">
     <origin xyz="0 0 0" rpy="0 0 0" />
   </xacro:VLP-16>

File: src/vehicle_simulator/urdf/rgbd_camera.urdf.xacro (robot description, xacro)
@@ -1,4 +1,4 @@
 <robot xmlns:xacro="http://www.ros.org/wiki/xacro" name="example">
-  <link name="camera">
+  <link name="rgbd_camera">
     <collision>
       <origin xyz="0 0 0" rpy="0 0 0"/>
@@ -19,32 +19,33 @@
     </inertial>
   </link>
-  <gazebo reference="camera">
-    <sensor type="camera" name="camera">
-      <update_rate>15.0</update_rate>
+  <gazebo reference="rgbd_camera">
+    <sensor type="depth" name="rgbd_camera">
+      <update_rate>30.0</update_rate>
+      <always_on>true</always_on>
       <camera name="head">
         <horizontal_fov>2.0</horizontal_fov>
         <image>
-          <width>320</width>
-          <height>180</height>
+          <width>640</width>
+          <height>360</height>
           <format>R8G8B8</format>
         </image>
         <clip>
           <near>0.1</near>
-          <far>200.0</far>
+          <far>30.0</far>
         </clip>
+        <distortion>
+          <k1>0.0</k1>
+          <k2>0.0</k2>
+          <k3>0.0</k3>
+          <p1>0.0</p1>
+          <p2>0.0</p2>
+        </distortion>
       </camera>
-      <plugin name="camera_controller" filename="libgazebo_ros_camera.so">
-        <alwaysOn>true</alwaysOn>
-        <updateRate>0.0</updateRate>
-        <cameraName>camera</cameraName>
-        <imageTopicName>image</imageTopicName>
-        <cameraInfoTopicName>camera_info</cameraInfoTopicName>
-        <frameName>camera</frameName>
-        <hackBaseline>0.0</hackBaseline>
-        <distortionK1>0.0</distortionK1>
-        <distortionK2>0.0</distortionK2>
-        <distortionK3>0.0</distortionK3>
-        <distortionT1>0.0</distortionT1>
-        <distortionT2>0.0</distortionT2>
+      <plugin name="rgbd_camera_controller" filename="libgazebo_ros_camera.so">
+          <baseline>0.2</baseline>
+          <camera_name>rgbd_camera</camera_name>
+          <frame_name>rgbd_camera</frame_name>
+          <min_depth>0.1</min_depth>
+          <pointCloudCutoffMax>30.0</pointCloudCutoffMax>
       </plugin>
     </sensor>
